File: hardware/logicboard/oao-001.sch (EAGLE design)
At the start: 9 parts, among them K1 G5V1, T1 2SC1815

Commit message: Released hardware.
Parts:
- removed J2: (no value), SparkFun-Connectors:CONN_02LOCK
- added D2: (no value), SparkFun-LED:LED-3MM-NO_SILK
- added R2: 220, resistor:R-US_0204/5
- added S3: NC: 5V, NO: 12V, SparkFun-Switches:SWITCH-SPDT-PTH-11.6X4.0MM
- added VIN: (no value), SparkFun-Connectors:CONN_02LOCK
- R1: value (none) -> 3.3k
- renumbered J1 to VOUT
Connections:
- new net N$13: R2.1, U$1.2
- new net N$14: D2.C, R2.2
- new net N$15: S3.S, U$1.9V
- net GND: now also VIN.2; no longer J2.2
- net VCC: now also D2.A, S3.O
- net VDD: now also S3.P, VIN.1; no longer J2.1, U$1.9V
Other:
- moved on the sheet: S1, S2

Commit message: Added capacitor.
Parts:
- added C1: (no value), capacitor-wima:C2,5-3
Connections:
- net GND: now also C1.2
- net VDD: now also C1.1
Changed lines of the file:
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@@
 <setting verticaltext="up"/>
 </settings>
-<grid distance="0.1" unitdist="inch" unit="inch" style="lines" multiple="1" display="yes" altdistance="0.01" altunitdist="inch" altunit="inch"/>
+<grid distance="0.1" unitdist="inch" unit="inch" style="lines" multiple="1" display="no" altdistance="0.01" altunitdist="inch" altunit="inch"/>
 <layers>
 <layer number="1" name="Top" color="4" fill="1" visible="no" active="no"/>
@@
 <part name="S3" library="SparkFun-Switches" deviceset="SWITCH-SPDT" device="-PTH-11.6X4.0MM" value="NC: 5V, NO: 12V"/>
 <part name="SUPPLY12" library="supply2" library_urn="urn:adsk.eagle:library:372" deviceset="VCC" device=""/>
+<part name="SUPPLY13" library="SparkFun-PowerSymbols" deviceset="VDD" device=""/>
+<part name="SUPPLY14" library="supply2" library_urn="urn:adsk.eagle:library:372" deviceset="GND" device=""/>
+<part name="C1" library="capacitor-wima" library_urn="urn:adsk.eagle:library:116" deviceset="C" device="2,5-3" package3d_urn="urn:adsk.eagle:package:5436/1"/>
 </parts>
 <sheets>
@@
 <instance part="S3" gate="1" x="38.1" y="30.48"/>
 <instance part="SUPPLY12" gate="G$1" x="45.72" y="40.64"/>
+<instance part="SUPPLY13" gate="VDD" x="127" y="33.02"/>
+<instance part="SUPPLY14" gate="GND" x="127" y="17.78"/>
+<instance part="C1" gate="G$1" x="127" y="27.94"/>
 </instances>
 <busses>
@@
 <pinref part="VIN" gate="G$1" pin="1"/>
 <wire x1="119.38" y1="78.74" x2="121.92" y2="78.74" width="0.1524" layer="91"/>
+</segment>
+<segment>
+<pinref part="C1" gate="G$1" pin="1"/>
+<pinref part="SUPPLY13" gate="VDD" pin="VDD"/>
+<wire x1="127" y1="33.02" x2="127" y2="30.48" width="0.1524" layer="91"/>
 </segment>
 </net>
@@
 <junction x="119.38" y="58.42"/>
 </segment>
+<segment>
+<pinref part="SUPPLY14" gate="GND" pin="GND"/>
+<pinref part="C1" gate="G$1" pin="2"/>
+<wire x1="127" y1="22.86" x2="127" y2="20.32" width="0.1524" layer="91"/>
+</segment>
 </net>

Commit message: GND.
Parts:
- removed S2: (no value), switch-dil:A1353HEX
- added OFF-INT: (no value), switch-dil:A1353HEX
- VOLTAGE-SELECT: value NC: 5V, NO: 12V -> 12V-5V
- renumbered D2 to LED, K1 to RELAY, S1 to ON-INT, S3 to VOLTAGE-SELECT
Connections:
- net N$13 renamed LEDDRIVE
- net N$15 renamed V12
- net N$2 renamed RELAYDRIVE
- removed net N$12: S2.1, U$1.4
- new net N$2: OFF-INT.8, U$1.8
- net GND: now also OFF-INT.C; no longer S2.C
- net N$11: now also OFF-INT.1; no longer S2.2
- net N$5: now also OFF-INT.4; no longer S2.8
- net N$6: now also OFF-INT.2; no longer S2.4
