File: hardware/logicboard/geyser-001.brd (EAGLE design)
At the start: 47 x 47 mm, 13 parts, among them T1 2SC1815

Commit message: Fixed missing silk pattern.
Parts:
- VIN, VOUT: device SparkFun-Connectors:JST-2-PTH-NS -> SparkFun-Connectors:JST-2-PTH
Changed lines of the file:
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@@
 <attribute name="VALUE" x="14.478" y="8.509" size="1.27" layer="27" ratio="10" rot="R90"/>
 </element>
-<element name="VOUT" library="SparkFun-Connectors" package="JST-2-PTH-NS" value="" x="6" y="10" smashed="yes" rot="R90">
+<element name="VOUT" library="SparkFun-Connectors" package="JST-2-PTH" value="" x="6" y="10" smashed="yes" rot="R90">
 <attribute name="NAME" x="6" y="6" size="0.8128" layer="25" font="vector" ratio="20" rot="R180" align="top-right"/>
+<attribute name="PROD_ID" value="CONN-09863" x="6" y="10" size="1.778" layer="27" rot="R90" display="off"/>
+<attribute name="SKU" value="PRT-09914" x="6" y="10" size="1.778" layer="27" rot="R90" display="off"/>
 <attribute name="VALUE" x="2" y="8.73" size="0.6096" layer="27" font="vector" ratio="20" rot="R90"/>
 </element>
-<element name="VIN" library="SparkFun-Connectors" package="JST-2-PTH-NS" value="" x="41" y="10" smashed="yes" rot="R270">
+<element name="VIN" library="SparkFun-Connectors" package="JST-2-PTH" value="" x="41" y="10" smashed="yes" rot="R270">
 <attribute name="NAME" x="39" y="6" size="0.6096" layer="25" font="vector" ratio="20"/>
+<attribute name="PROD_ID" value="CONN-09863" x="41" y="10" size="1.778" layer="27" rot="R270" display="off"/>
+<attribute name="SKU" value="PRT-09914" x="41" y="10" size="1.778" layer="27" rot="R270" display="off"/>
 <attribute name="VALUE" x="45" y="11.27" size="0.6096" layer="27" font="vector" ratio="20" rot="R270"/>
 </element>
