File: hardware/logicboard/geyser-001.sch (EAGLE design)
At the start: 13 parts, among them T1 2SC1815

Commit message: Added silk.
Connections:
- net V12 renamed VIN
Changed lines of the file:
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@@
 </segment>
 </net>
-<net name="V12" class="0">
+<net name="VIN" class="0">
 <segment>
 <pinref part="VOLTAGE-SELECT" gate="1" pin="S"/>

Commit message: Changed copyright notice.
Other:
- note added: "Geyser 1.0.0 by Pineapple Design"
Changed lines of the file:
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@@
 <sheet>
 <plain>
+<text x="22.86" y="15.24" size="1.778" layer="91">Geyser 1.0.0 by Pineapple Design</text>
 </plain>
 <instances>

Commit message: New layout.
Parts:
- C1: value (none) -> 104
- D1: value 1N4004 -> 200mA/100V/1V; device diode:1N4004 -> SparkFun-DiscreteSemi:DIODE-1N4148
- VIN, VOUT: device SparkFun-Connectors:CONN_02LOCK -> SparkFun-Connectors:CONN_02-JST-2-PTH-NO_SILK
Connections:
- removed net N$1: RELAY2.P, VOUT.1
- new net VOUT: RELAY2.P, VOUT.2
- net GND: now also VIN.1, VOUT.1; no longer VIN.2, VOUT.2
- net VDD: now also VIN.2; no longer VIN.1
Other:
- moved on the sheet: VIN, VOUT
Changed lines of the file:
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@@
 <clearance class="0" value="0.254"/>
+</class>
+<class number="1" name="VDD" width="0.254" drill="0.127">
+<clearance class="1" value="0.254"/>
+</class>
+<class number="2" name="VOUT" width="0.254" drill="0.127">
+<clearance class="2" value="0.254"/>
 </class>
 </classes>
@@
 <part name="SUPPLY3" library="SparkFun-PowerSymbols" deviceset="VDD" device=""/>
 <part name="SUPPLY4" library="supply2" library_urn="urn:adsk.eagle:library:372" deviceset="GND" device=""/>
-<part name="VOUT" library="SparkFun-Connectors" deviceset="CONN_02" device="LOCK"/>
 <part name="SUPPLY5" library="supply2" library_urn="urn:adsk.eagle:library:372" deviceset="GND" device=""/>
 <part name="R1" library="resistor" library_urn="urn:adsk.eagle:library:348" deviceset="R-US_" device="0204/5" package3d_urn="urn:adsk.eagle:package:25955/1" value="3.3k"/>
@@
 <part name="SUPPLY7" library="supply2" library_urn="urn:adsk.eagle:library:372" deviceset="VCC" device=""/>
 <part name="SUPPLY8" library="supply2" library_urn="urn:adsk.eagle:library:372" deviceset="VCC" device=""/>
-<part name="D1" library="diode" library_urn="urn:adsk.eagle:library:210" deviceset="1N4004" device="" package3d_urn="urn:adsk.eagle:package:43336/1"/>
+<part name="D1" library="SparkFun-DiscreteSemi" deviceset="DIODE" device="-1N4148" value="200mA/100V/1V"/>
 <part name="ON-INT" library="switch-dil" library_urn="urn:adsk.eagle:library:375" deviceset="A1353HEX" device="" package3d_urn="urn:adsk.eagle:package:27207/1"/>
 <part name="OFF-INT" library="switch-dil" library_urn="urn:adsk.eagle:library:375" deviceset="A1353HEX" device="" package3d_urn="urn:adsk.eagle:package:27207/1"/>
 <part name="SUPPLY9" library="supply2" library_urn="urn:adsk.eagle:library:372" deviceset="GND" device=""/>
-<part name="VIN" library="SparkFun-Connectors" deviceset="CONN_02" device="LOCK"/>
 <part name="SUPPLY10" library="SparkFun-PowerSymbols" deviceset="VDD" device=""/>
 <part name="R2" library="resistor" library_urn="urn:adsk.eagle:library:348" deviceset="R-US_" device="0204/5" package3d_urn="urn:adsk.eagle:package:25955/1" value="220"/>
@@
 <part name="SUPPLY13" library="SparkFun-PowerSymbols" deviceset="VDD" device=""/>
 <part name="SUPPLY14" library="supply2" library_urn="urn:adsk.eagle:library:372" deviceset="GND" device=""/>
-<part name="C1" library="capacitor-wima" library_urn="urn:adsk.eagle:library:116" deviceset="C" device="2,5-3" package3d_urn="urn:adsk.eagle:package:5436/1"/>
+<part name="C1" library="capacitor-wima" library_urn="urn:adsk.eagle:library:116" deviceset="C" device="2,5-3" package3d_urn="urn:adsk.eagle:package:5436/1" value="104"/>
+<part name="VOUT" library="SparkFun-Connectors" deviceset="CONN_02" device="-JST-2-PTH-NO_SILK"/>
+<part name="VIN" library="SparkFun-Connectors" deviceset="CONN_02" device="-JST-2-PTH-NO_SILK"/>
 </parts>
 <sheets>
@@
 <instance part="SUPPLY3" gate="VDD" x="43.18" y="91.44"/>
 <instance part="SUPPLY4" gate="GND" x="43.18" y="53.34"/>
-<instance part="VOUT" gate="G$1" x="22.86" y="78.74" rot="MR180"/>
 <instance part="SUPPLY5" gate="GND" x="33.02" y="53.34"/>
 <instance part="R1" gate="G$1" x="63.5" y="63.5"/>
@@
 <instance part="SUPPLY7" gate="G$1" x="50.8" y="91.44"/>
 <instance part="SUPPLY8" gate="G$1" x="66.04" y="40.64"/>
-<instance part="D1" gate="1" x="60.96" y="78.74" rot="R90"/>
+<instance part="D1" gate="G$1" x="60.96" y="78.74" rot="R90"/>
 <instance part="ON-INT" gate="1" x="109.22" y="58.42" rot="R90"/>
 <instance part="OFF-INT" gate="1" x="109.22" y="48.26" rot="R90"/>
 <instance part="SUPPLY9" gate="GND" x="119.38" y="17.78"/>
-<instance part="VIN" gate="G$1" x="129.54" y="78.74" rot="R180"/>
 <instance part="SUPPLY10" gate="VDD" x="119.38" y="91.44"/>
 <instance part="R2" gate="G$1" x="99.06" y="71.12" rot="R90"/>
@@
 <instance part="SUPPLY14" gate="GND" x="127" y="17.78"/>
 <instance part="C1" gate="G$1" x="127" y="27.94"/>
+<instance part="VOUT" gate="G$1" x="22.86" y="76.2"/>
+<instance part="VIN" gate="G$1" x="109.22" y="76.2"/>
 </instances>
 <busses>
@@
 </segment>
 <segment>
-<pinref part="SUPPLY10" gate="VDD" pin="VDD"/>
-<wire x1="119.38" y1="91.44" x2="119.38" y2="78.74" width="0.1524" layer="91"/>
-<pinref part="VIN" gate="G$1" pin="1"/>
-<wire x1="119.38" y1="78.74" x2="121.92" y2="78.74" width="0.1524" layer="91"/>
-</segment>
-<segment>
 <pinref part="C1" gate="G$1" pin="1"/>
 <pinref part="SUPPLY13" gate="VDD" pin="VDD"/>
 <wire x1="127" y1="33.02" x2="127" y2="30.48" width="0.1524" layer="91"/>
+</segment>
+<segment>
+<wire x1="116.84" y1="78.74" x2="119.38" y2="78.74" width="0.1524" layer="91"/>
+<pinref part="VIN" gate="G$1" pin="2"/>
+<pinref part="SUPPLY10" gate="VDD" pin="VDD"/>
+<wire x1="119.38" y1="91.44" x2="119.38" y2="78.74" width="0.1524" layer="91"/>
 </segment>
 </net>
@@
 </segment>
 <segment>
-<pinref part="VOUT" gate="G$1" pin="2"/>
 <pinref part="SUPPLY5" gate="GND" pin="GND"/>
 <wire x1="30.48" y1="76.2" x2="33.02" y2="76.2" width="0.1524" layer="91"/>
 <wire x1="33.02" y1="76.2" x2="33.02" y2="55.88" width="0.1524" layer="91"/>
+<pinref part="VOUT" gate="G$1" pin="1"/>
 </segment>
 <segment>
@@
 <wire x1="119.38" y1="20.32" x2="119.38" y2="48.26" width="0.1524" layer="91"/>
 <junction x="119.38" y="48.26"/>
-<pinref part="VIN" gate="G$1" pin="2"/>
-<wire x1="121.92" y1="76.2" x2="119.38" y2="76.2" width="0.1524" layer="91"/>
-<wire x1="119.38" y1="76.2" x2="119.38" y2="58.42" width="0.1524" layer="91"/>
+<pinref part="VIN" gate="G$1" pin="1"/>
+<wire x1="119.38" y1="76.2" x2="116.84" y2="76.2" width="0.1524" layer="91"/>
+<wire x1="119.38" y1="58.42" x2="119.38" y2="76.2" width="0.1524" layer="91"/>
 <junction x="119.38" y="58.42"/>
 </segment>
@@
 </segment>
 </net>
-<net name="N$1" class="0">
+<net name="VOUT" class="0">
 <segment>
 <pinref part="RELAY" gate="2" pin="P"/>
-<pinref part="VOUT" gate="G$1" pin="1"/>
 <wire x1="35.56" y1="78.74" x2="30.48" y2="78.74" width="0.1524" layer="91"/>
+<pinref part="VOUT" gate="G$1" pin="2"/>
 </segment>
 </net>
@@
 <pinref part="RELAY" gate="1" pin="2"/>
 <wire x1="50.8" y1="73.66" x2="50.8" y2="71.12" width="0.1524" layer="91"/>
-<pinref part="D1" gate="1" pin="A"/>
+<pinref part="D1" gate="G$1" pin="A"/>
 <wire x1="50.8" y1="71.12" x2="50.8" y2="68.58" width="0.1524" layer="91"/>
 <wire x1="60.96" y1="76.2" x2="60.96" y2="71.12" width="0.1524" layer="91"/>
@@
 <pinref part="RELAY" gate="1" pin="1"/>
 <wire x1="50.8" y1="88.9" x2="50.8" y2="86.36" width="0.1524" layer="91"/>
-<pinref part="D1" gate="1" pin="C"/>
+<pinref part="D1" gate="G$1" pin="C"/>
 <wire x1="50.8" y1="86.36" x2="50.8" y2="83.82" width="0.1524" layer="91"/>
 <wire x1="60.96" y1="81.28" x2="60.96" y2="86.36" width="0.1524" layer="91"/>

Commit message: Swapped + and -. Now + is on No.1 pin.
Parts:
- R2: value 220 -> 330
Connections:
- net GND: now also VOUT.2; no longer VOUT.1
- net VOUT: now also VOUT.1; no longer VOUT.2
Other:
- moved on the sheet: VIN, VOUT
Changed lines of the file:
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@@
 <?xml version="1.0" encoding="utf-8"?>
 <!DOCTYPE eagle SYSTEM "eagle.dtd">
-<eagle version="8.6.3">
+<eagle version="8.7.0">
 <drawing>
 <settings>
@@
 <clearance class="0" value="0.254"/>
 </class>
-<class number="1" name="VDD" width="0.254" drill="0.127">
-<clearance class="1" value="0.254"/>
-</class>
-<class number="2" name="VOUT" width="0.254" drill="0.127">
-<clearance class="2" value="0.254"/>
-</class>
 </classes>
 <parts>
@@
 <part name="SUPPLY9" library="supply2" library_urn="urn:adsk.eagle:library:372" deviceset="GND" device=""/>
 <part name="SUPPLY10" library="SparkFun-PowerSymbols" deviceset="VDD" device=""/>
-<part name="R2" library="resistor" library_urn="urn:adsk.eagle:library:348" deviceset="R-US_" device="0204/5" package3d_urn="urn:adsk.eagle:package:25955/1" value="220"/>
+<part name="R2" library="resistor" library_urn="urn:adsk.eagle:library:348" deviceset="R-US_" device="0204/5" package3d_urn="urn:adsk.eagle:package:25955/1" value="330"/>
 <part name="LED" library="SparkFun-LED" deviceset="LED" device="-3MM-NO_SILK"/>
 <part name="SUPPLY11" library="supply2" library_urn="urn:adsk.eagle:library:372" deviceset="VCC" device=""/>
@@
 <instance part="SUPPLY14" gate="GND" x="127" y="17.78"/>
 <instance part="C1" gate="G$1" x="127" y="27.94"/>
-<instance part="VOUT" gate="G$1" x="22.86" y="76.2"/>
-<instance part="VIN" gate="G$1" x="109.22" y="76.2"/>
+<instance part="VOUT" gate="G$1" x="22.86" y="78.74" rot="MR180"/>
+<instance part="VIN" gate="G$1" x="129.54" y="76.2" rot="MR0"/>
 </instances>
 <busses>
@@
 </segment>
 <segment>
-<wire x1="116.84" y1="78.74" x2="119.38" y2="78.74" width="0.1524" layer="91"/>
-<pinref part="VIN" gate="G$1" pin="2"/>
 <pinref part="SUPPLY10" gate="VDD" pin="VDD"/>
 <wire x1="119.38" y1="91.44" x2="119.38" y2="78.74" width="0.1524" layer="91"/>
+<pinref part="VIN" gate="G$1" pin="2"/>
+<wire x1="121.92" y1="78.74" x2="119.38" y2="78.74" width="0.1524" layer="91"/>
 </segment>
 </net>
@@
 <segment>
 <pinref part="SUPPLY5" gate="GND" pin="GND"/>
+<wire x1="33.02" y1="76.2" x2="33.02" y2="55.88" width="0.1524" layer="91"/>
+<pinref part="VOUT" gate="G$1" pin="2"/>
 <wire x1="30.48" y1="76.2" x2="33.02" y2="76.2" width="0.1524" layer="91"/>
-<wire x1="33.02" y1="76.2" x2="33.02" y2="55.88" width="0.1524" layer="91"/>
-<pinref part="VOUT" gate="G$1" pin="1"/>
 </segment>
 <segment>
@@
 <wire x1="119.38" y1="20.32" x2="119.38" y2="48.26" width="0.1524" layer="91"/>
 <junction x="119.38" y="48.26"/>
-<pinref part="VIN" gate="G$1" pin="1"/>
-<wire x1="119.38" y1="76.2" x2="116.84" y2="76.2" width="0.1524" layer="91"/>
 <wire x1="119.38" y1="58.42" x2="119.38" y2="76.2" width="0.1524" layer="91"/>
 <junction x="119.38" y="58.42"/>
+<pinref part="VIN" gate="G$1" pin="1"/>
+<wire x1="121.92" y1="76.2" x2="119.38" y2="76.2" width="0.1524" layer="91"/>
 </segment>
 <segment>
@@
 <pinref part="C1" gate="G$1" pin="2"/>
 <wire x1="127" y1="22.86" x2="127" y2="20.32" width="0.1524" layer="91"/>
-</segment>
-</net>
-<net name="VOUT" class="0">
-<segment>
-<pinref part="RELAY" gate="2" pin="P"/>
-<wire x1="35.56" y1="78.74" x2="30.48" y2="78.74" width="0.1524" layer="91"/>
-<pinref part="VOUT" gate="G$1" pin="2"/>
 </segment>
 </net>
@@
 </segment>
 </net>
+<net name="VOUT" class="0">
+<segment>
+<pinref part="RELAY" gate="2" pin="P"/>
+<pinref part="VOUT" gate="G$1" pin="1"/>
+<wire x1="35.56" y1="78.74" x2="30.48" y2="78.74" width="0.1524" layer="91"/>
+</segment>
+</net>

Commit message: Fixed missing silk pattern.
Parts:
- VIN, VOUT: device SparkFun-Connectors:CONN_02-JST-2-PTH-NO_SILK -> SparkFun-Connectors:CONN_02JST-PTH-2
Changed lines of the file:
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@@
 <setting verticaltext="up"/>
 </settings>
-<grid distance="0.1" unitdist="inch" unit="inch" style="lines" multiple="1" display="yes" altdistance="0.01" altunitdist="inch" altunit="inch"/>
+<grid distance="0.1" unitdist="inch" unit="inch" style="lines" multiple="1" display="no" altdistance="0.01" altunitdist="inch" altunit="inch"/>
 <layers>
 <layer number="1" name="Top" color="4" fill="1" visible="no" active="no"/>
@@
 <part name="SUPPLY14" library="supply2" library_urn="urn:adsk.eagle:library:372" deviceset="GND" device=""/>
 <part name="C1" library="capacitor-wima" library_urn="urn:adsk.eagle:library:116" deviceset="C" device="2,5-3" package3d_urn="urn:adsk.eagle:package:5436/1" value="104"/>
-<part name="VOUT" library="SparkFun-Connectors" deviceset="CONN_02" device="-JST-2-PTH-NO_SILK"/>
-<part name="VIN" library="SparkFun-Connectors" deviceset="CONN_02" device="-JST-2-PTH-NO_SILK"/>
+<part name="VOUT" library="SparkFun-Connectors" deviceset="CONN_02" device="JST-PTH-2"/>
+<part name="VIN" library="SparkFun-Connectors" deviceset="CONN_02" device="JST-PTH-2"/>
 </parts>
 <sheets>
